File: HRU-SCB-RP2040/servo_serial.kicad_sch (KiCad schematic)
At the start: 16 parts, among them U5 SN65HVD11HD, U6 SN65HVD11HD

Commit message: Delete PWM circuit
Parts:
- removed Q? (x4): BSS138, Package_TO_SOT_SMD:SOT-23, symbol Transistor_FET:BSS138
- removed RN8, RN9, RN? (x8): 2.2k, Resistor_SMD:R_Array_Convex_4x1206, symbol Device:R_Pack04_Split
- removed U5, U6: SN65HVD11HD, Package_SO:SOIC-8_3.9x4.9mm_P1.27mm, symbol Interface_UART:SN65HVD11HD
Connections:
- no-connect marks 4 -> 0
