File: HRU-SCB-uHAT/HRU-SCB-uHAT.kicad_sch (KiCad schematic)
At the start: 22 parts, among them J1 GPIO, J2 Conn_01x03_Pin, J3 Conn_01x03_Pin, J4 Conn_01x03_Pin, J5 Conn_01x03_Pin, J6 Conn_01x03_Pin, J7 Conn_01x03_Pin, J8 Conn_01x03_Pin, J9 Conn_01x03_Pin, U1 CAT24C256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

Commit message: Update: fix parts layout
Parts:
- removed J2, J3, J4, J5, J6, J7, J8, J9: Conn_01x03_Pin, symbol Connector:Conn_01x03_Pin
- removed JP1: ID_WP, symbol Jumper:SolderJumper_2_Open
- removed U1: CAT24C256, symbol Memory_EEPROM:CAT24C256
- removed U2: SC16IS762IPW, Package_SO:TSSOP-28_4.4x9.7mm_P0.65mm, symbol Interface_UART:SC16IS762IPW
- removed U3, U4: 74AHCT2G241, Package_SO:VSSOP-8_2.3x2mm_P0.5mm, symbol 74xGxx:74AUC2G241
- removed Y1: Crystal_GND24_Small, symbol Device:Crystal_GND24_Small
- added C3, C4, C5: 1.0u, Capacitor_SMD:C_0603_1608Metric_Pad1.08x0.95mm_HandSolder, symbol Device:C_Small
- added R6: 10k, Resistor_SMD:R_0603_1608Metric_Pad0.98x0.95mm_HandSolder, symbol Device:R_Small
- added U1: MAX14830, Package_DFN_QFN:TQFN-48-1EP_7x7mm_P0.5mm_EP5.1x5.1mm, symbol Interface_UART:MAX14830
- added Y1: FA-238 16.0000MB-C3, Crystal:Crystal_SMD_3225-4Pin_3.2x2.5mm_HandSoldering, symbol Device:Crystal_GND24
- C1: value 100n -> 1.0u; footprint (none) -> Capacitor_SMD:C_0603_1608Metric_Pad1.08x0.95mm_HandSolder
- C2: value C_Small -> 10u; footprint (none) -> Capacitor_SMD:C_0603_1608Metric_Pad1.08x0.95mm_HandSolder
- J3: renamed from J1; footprint Connector_PinSocket_2.54mm:PinSocket_2x20_P2.54mm_Vertical -> Connector_PinSocket_2.54mm:PinSocket_2x20_P2.54mm_Vertical_SMD
- R1, R2: value 3.9k -> 2.2k; footprint (none) -> Resistor_SMD:R_0603_1608Metric_Pad0.98x0.95mm_HandSolder
- R3, R4, R5: value 1k -> 10k; footprint (none) -> Resistor_SMD:R_0603_1608Metric_Pad0.98x0.95mm_HandSolder
Connections:
- net +3V3: now also C2.1, R3.1, C3.1, C4.1, U1.2 (LDOEN), U1.43 (VEXT), U1.47 (VA), U1.9 (VL)
- net +5V: now also R5.1
- net GND: now also C2.2, C3.2, C4.2, C5.1, R6.2, U1.10 (DGND), U1.46 (AGND), U1.49 (AGND), Y1.2, Y1.4; no longer R5.2
- net GPIO10/SPI0.MOSI: now also U1.6 (MOSI/A1)
- net GPIO11/SPI0.SCLK: now also U1.4 (SCLK/SCL)
- net GPIO24: no longer R3.2
- net GPIO27: now also R1.2, U1.7 (~{IRQ})
- net GPIO8/SPI0.CE0: now also U1.5 (~{CS}/A0)
- net GPIO9/SPI0.MISO: now also U1.3 (MISO/SDA)
- net ID_SCL: no longer R2.2
- net ID_SDA: no longer R1.2
- net at R4.1: now also U1.16 (~{CTS0}), U1.24 (~{CTS1}), U1.32 (~{CTS2}), U1.40 (~{CTS3})
- new net: C5.2, U1.48 (V18)
- new net: R3.2, U1.1 (SPI/~{I2C})
- new net: U1.44 (XOUT), Y1.1
- new net: U1.45 (XIN), Y1.3
- new net: R2.2, U1.8 (~{RST})
- new net ServoDriver0/2.5V: R5.2, R6.1
- new net ServoDriver0/SERIAL.RX: U1.17 (RX0)
- new net ServoDriver0/SERIAL.TX: U1.18 (TX0)
- new net ServoDriver0/SERIAL.~{EN}: U1.15 (~{RTS0})
- new net ServoDriver1/SERIAL.RX: U1.25 (RX1)
- new net ServoDriver1/SERIAL.TX: U1.26 (TX1)
- new net ServoDriver1/SERIAL.~{EN}: U1.23 (~{RTS1})
- new net ServoDriver2/SERIAL.RX: U1.33 (RX2)
- new net ServoDriver2/SERIAL.TX: U1.34 (TX2)
- new net ServoDriver2/SERIAL.~{EN}: U1.31 (~{RTS2})
- new net ServoDriver3/SERIAL.RX: U1.41 (RX3)
- new net ServoDriver3/SERIAL.TX: U1.42 (TX3)
- new net ServoDriver3/SERIAL.~{EN}: U1.39 (~{RTS3})
- no-connect marks 12 -> 16
Other:
- added sheet ExtendConnector (extend_connector.kicad_sch)
- added sheet ServoConnector0 (servo_connector_typeA.kicad_sch)
- added sheet ServoConnector1 (servo_connector_typeB.kicad_sch)
- added sheet ServoConnector2 (servo_connector_typeB.kicad_sch)
- added sheet ServoConnector3 (servo_connector_typeA.kicad_sch)
- added sheet ServoDriver0 (servo_driver.kicad_sch)
- added sheet ServoDriver1 (servo_driver.kicad_sch)
- added sheet ServoDriver2 (servo_driver.kicad_sch)
- added sheet ServoDriver3 (servo_driver.kicad_sch)
- note added: "https://github.com/analogdevicesinc/linux/blob/rpi-5.10.y/arch/arm/boot/dts/overlays/rpi-max14830-spi-overlay.dts"
- note removed: "ID_SD and ID_SC PINS: These pins are reserved for HAT ID EEPROM. At boot time this I2C interface will be interrogated to look for an EEPROM that identifes the attached board and allows automagic setup of the GPIOs (and optionally, Linux drivers). Bridging JP1 enables write protection. DO NOT USE these pins for anything other than attaching an I2C ID EEPROM. Leave unconnected if ID EEPROM not requ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"
- moved on the sheet: R4

Commit message: Update: fix ERC error
Connections:
- no-connect marks 16 -> 33
Changed lines of the file:
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@@
 	)
 	(no_connect
+		(at 95.25 71.12)
+	)
+	(no_connect
+		(at 26.67 45.72)
+	)
+	(no_connect
 		(at 180.34 127)
 	)
 	(no_connect
+		(at 26.67 40.64)
+	)
+	(no_connect
 		(at 180.34 55.88)
 	)
 	(no_connect
+		(at 95.25 58.42)
+	)
+	(no_connect
+		(at 26.67 63.5)
+	)
+	(no_connect
+		(at 95.25 60.96)
+	)
+	(no_connect
 		(at 180.34 106.68)
 	)
 	(no_connect
+		(at 26.67 35.56)
+	)
+	(no_connect
 		(at 180.34 101.6)
 	)
 	(no_connect
+		(at 26.67 71.12)
+	)
+	(no_connect
+		(at 95.25 76.2)
+	)
+	(no_connect
+		(at 95.25 48.26)
+	)
+	(no_connect
+		(at 26.67 73.66)
+	)
+	(no_connect
 		(at 180.34 76.2)
 	)
 	(no_connect
+		(at 95.25 45.72)
+	)
+	(no_connect
 		(at 180.34 121.92)
 	)
 	(no_connect
+		(at 95.25 53.34)
+	)
+	(no_connect
+		(at 26.67 60.96)
+	)
+	(no_connect
 		(at 180.34 60.96)
 	)
 	(no_connect
+		(at 95.25 40.64)
+	)
+	(no_connect
 		(at 180.34 104.14)
 	)
@@
 	)
 	(no_connect
+		(at 95.25 73.66)
+	)
+	(no_connect
 		(at 180.34 78.74)
 	)
@@
 		(at 180.34 124.46)
 	)
+	(no_connect
+		(at 26.67 66.04)
+	)
 	(wire
 		(pts
@@
 	(wire
 		(pts
+			(xy 38.1 27.94) (xy 50.8 27.94)
+		)
+		(stroke
+			(width 0)
+			(type default)
+		)
+	)
+	(wire
+		(pts
 			(xy 147.32 114.3) (xy 149.86 114.3)
 		)
@@
 	(wire
 		(pts
+			(xy 38.1 24.13) (xy 38.1 27.94)
+		)
+		(stroke
+			(width 0)
+			(type default)
+		)
+	)
+	(wire
+		(pts
 			(xy 101.6 104.14) (xy 114.3 104.14)
 		)
@@
 					(size 1.27 1.27)
 				)
+				(hide yes)
 			)
 		)
@@
 					(size 1.27 1.27)
 				)
+				(hide yes)
 			)
 		)
-		(property "Description" ""
+		(property "Description" "Power symbol creates a global label with name \"+5V\""
 			(at 71.12 24.13 0)
 			(effects
@@
 					(size 1.27 1.27)
 				)
+				(hide yes)
 			)
 		)
@@
 					(size 1.27 1.27)
 				)
+				(hide yes)
 			)
 		)
-		(property "Description" ""
+		(property "Description" "Power symbol creates a global label with name \"+3.3V\""
 			(at 50.8 24.13 0)
 			(effects
@@
 					(size 1.27 1.27)
 				)
+				(hide yes)
 			)
 		)
@@
 					(size 1.27 1.27)
 				)
+				(hide yes)
 			)
 		)
-		(property "Description" ""
+		(property "Description" "Power symbol creates a global label with name \"GND\" , ground"
 			(at 71.12 80.01 0)
 			(effects
@@
 					(size 1.27 1.27)
 				)
+				(hide yes)
 			)
 		)
@@
 					(size 1.27 1.27)
 				)
+				(hide yes)
 			)
 		)
-		(property "Description" ""
+		(property "Description" "Power symbol creates a global label with name \"GND\" , ground"
 			(at 53.34 80.01 0)
 			(effects
@@
 	)
 	(symbol
+		(lib_name "R_Small_1")
 		(lib_id "Device:R_Small")
 		(at 226.06 38.1 90)
@@
 	)
 	(symbol
-		(lib_name "GND_1")
 		(lib_id "power:GND")
 		(at 165.1 152.4 0)
@@
 	)
 	(symbol
-		(lib_name "GND_1")
 		(lib_id "power:GND")
 		(at 231.14 40.64 0)
@@
 	)
 	(symbol
-		(lib_name "GND_1")
+		(lib_id "power:PWR_FLAG")
+		(at 38.1 24.13 0)
+		(unit 1)
+		(exclude_from_sim no)
+		(in_bom yes)
+		(on_board yes)
+		(dnp no)
+		(fields_autoplaced yes)
+		(property "Reference" "#FLG03"
+			(at 38.1 22.225 0)
+			(effects
+				(font
+					(size 1.27 1.27)
+				)
+				(hide yes)
+			)
+		)
+		(property "Value" "PWR_FLAG"
+			(at 38.1 19.05 0)
+			(effects
+				(font
+					(size 1.27 1.27)
+				)
+			)
+		)
+		(property "Footprint" ""
+			(at 38.1 24.13 0)
+			(effects
+				(font
+					(size 1.27 1.27)
+				)
+				(hide yes)
+			)
+		)
+		(property "Datasheet" "~"
+			(at 38.1 24.13 0)
+			(effects
+				(font
+					(size 1.27 1.27)
+				)
+				(hide yes)
+			)
+		)
+		(property "Description" "Special symbol for telling ERC where power comes from"
+			(at 38.1 24.13 0)
+			(effects
+				(font
+					(size 1.27 1.27)
+				)
+				(hide yes)
+			)
+		)
+		(pin "1"
+		)
+		(instances
+			(project ""
+				(path "/e63e39d7-6ac0-4ffd-8aa3-1841a4541b55"
+					(reference "#FLG03")
+					(unit 1)
+				)
+			)
+		)
+	)
+	(symbol
 		(lib_id "power:GND")
 		(at 167.64 38.1 0)
@@
 	)
 	(symbol
+		(lib_name "R_Small_4")
 		(lib_id "Device:R_Small")
 		(at 114.3 96.52 0)
@@
 					(size 1.27 1.27)
 				)
+				(hide yes)
 			)
 		)
@@
 					(size 1.27 1.27)
 				)
+				(hide yes)
 			)
 		)
-		(property "Description" ""
+		(property "Description" "Power symbol creates a global label with name \"+3.3V\""
 			(at 121.92 91.44 0)
 			(effects
@@
 					(size 1.27 1.27)
 				)
+				(hide yes)
 			)
 		)
@@
 					(size 1.27 1.27)
 				)
+				(hide yes)
 			)
 		)
-		(property "Description" ""
+		(property "Description" "Power symbol creates a global label with name \"+3.3V\""
 			(at 160.02 25.4 0)
 			(effects
@@
 					(size 1.27 1.27)
 				)
+				(hide yes)
 			)
 		)
@@
 					(size 1.27 1.27)
 				)
+				(hide yes)
 			)
 		)
-		(property "Description" ""
+		(property "Description" "Power symbol creates a global label with name \"+3.3V\""
 			(at 152.4 25.4 0)
 			(effects
@@
 	)
 	(symbol
-		(lib_name "GND_1")
 		(lib_id "power:GND")
 		(at 160.02 38.1 0)
@@
 	)
 	(symbol
+		(lib_name "R_Small_3")
 		(lib_id "Device:R_Small")
 		(at 215.9 38.1 90)
@@
 	)
 	(symbol
+		(lib_name "R_Small_2")
 		(lib_id "Device:R_Small")
 		(at 121.92 96.52 0)
@@
 					(size 1.27 1.27)
 				)
+				(hide yes)
 			)
 		)
@@
 					(size 1.27 1.27)
 				)
+				(hide yes)
 			)
 		)
-		(property "Description" ""
+		(property "Description" "Power symbol creates a global label with name \"+3.3V\""
 			(at 167.64 25.4 0)
 			(effects
@@
 	)
 	(symbol
-		(lib_name "GND_1")
 		(lib_id "power:GND")
 		(at 187.96 38.1 0)
@@
 					(size 1.27 1.27)
 				)
+				(hide yes)
 			)
 		)
@@
 					(size 1.27 1.27)
 				)
+				(hide yes)
 			)
 		)
-		(property "Description" ""
+		(property "Description" "Power symbol creates a global label with name \"+3.3V\""
 			(at 114.3 91.44 0)
 			(effects
@@
 	)
 	(symbol
-		(lib_name "GND_1")
 		(lib_id "power:GND")
 		(at 139.7 68.58 0)
@@
 					(size 1.27 1.27)
 				)
+				(hide yes)
 			)
 		)
@@
 					(size 1.27 1.27)
 				)
+				(hide yes)
 			)
 		)
-		(property "Description" ""
+		(property "Description" "Power symbol creates a global label with name \"+3.3V\""
 			(at 147.32 78.74 0)
 			(effects
@@
 	)
 	(symbol
-		(lib_name "GND_1")
 		(lib_id "power:GND")
 		(at 127 129.54 0)
@@
 	)
 	(symbol
+		(lib_name "R_Small_5")
 		(lib_id "Device:R_Small")
 		(at 147.32 83.82 0)
@@
 	)
 	(symbol
-		(lib_name "GND_1")
 		(lib_id "power:GND")
 		(at 144.78 38.1 0)
@@
 					(size 1.27 1.27)
 				)
+				(hide yes)
 			)
 		)
@@
 					(size 1.27 1.27)
 				)
+				(hide yes)
 			)
 		)
-		(property "Description" ""
+		(property "Description" "Power symbol creates a global label with name \"+3.3V\""
 			(at 139.7 55.88 0)
 			(effects
