File: HRU-SCB-uHAT/extend_connector.kicad_sch (KiCad schematic)
At the start: 13 parts, among them J1 Conn_01x02_Pin, J2 Conn_01x02_MountingPin, J4 GROVE-CONNECTOR-SMD_4+2P-2.0_, J5 GROVE-CONNECTOR-SMD_4+2P-2.0_, J6 Conn_01x03_Pin

Commit message: Update: fix ERC error
Connections:
- net GND: now also J4.SS1, J4.SS2, J5.SS1, J5.SS2; no longer J4.5 (SS1), J4.6 (SS2), J5.5 (SS1), J5.6 (SS2)
- net +3.3V renamed +3V3
