File: HRU-SCB-M5Atom-Entry/servo_serial.kicad_sch (KiCad schematic)
At the start: 6 parts, among them Q1 BS170, U3 MAX485E

Commit message: Update: PCB wires
Parts:
- Q1: AKI_CODE (none) -> 109724; AKI_URL (none) -> https://akizukidenshi.com/catalog/g/g109724/
- R3, R4, R5: AKI_CODE (none) -> 125222; AKI_URL (none) -> https://akizukidenshi.com/catalog/g/g125222/
- U3: AKI_CODE (none) -> 115806; AKI_URL (none) -> https://akizukidenshi.com/catalog/g/g115806/
